File: Controlexp/Controlexp.kicad_sch (KiCad schematic)
At the start: 26 parts, among them J1 SMA_CONNECTOR, J4 530470510, J5 Power Connector, J6 Pressure sensor, J7 POWER PROBE, U2 RFM95W, U3 TPS62162DSG, U4 BME680, U5 XIAO-nRF52840-DIP

Commit message: fresh board
Parts:
- removed H1: GND, MountingHole:MountingHole_2.5mm_Pad, symbol Mechanical:MountingHole_Pad
- removed H2: 12V, MountingHole:MountingHole_2.5mm_Pad, symbol Mechanical:MountingHole_Pad
- removed J1: SMA_CONNECTOR, SMASMA2:CONN_RF2-04A-T-00-50-G_ADM, symbol SMA_Connector:SMA_CONNECTOR
- removed J7: POWER PROBE, Connector_PinHeader_2.54mm:PinHeader_1x03_P2.54mm_Vertical, symbol Connector_Generic:Conn_01x03
- removed U5: XIAO-nRF52840-DIP, MCU_SEED:MODULE_113991054, symbol MCU_SEEED_XIAO_Series:XIAO-nRF52840-DIP
- added C10, C9: 220 uF, Capacitor_SMD:C_0805_2012Metric, symbol Device:C_Small
- added C11: 10uF, 25V, Capacitor_SMD:C_0805_2012Metric, symbol Device:C_Small
- added C12: 22uF, 10V, Capacitor_SMD:C_0805_2012Metric, symbol Device:C_Small
- added C13, C14: 100nF, Capacitor_SMD:C_0805_2012Metric, symbol Device:C
- added D2: SS34, SS34:DIOM7959X265N, symbol SS34:SS34
- added J1: Conn_Coaxial_Small, SMAv2:CONN_RF2-04A-T-00-50-G_ADM, symbol Connector:Conn_Coaxial_Small
- added J10: Extra sensor TOP, Connector_JST:JST_GH_BM04B-GHS-TBT_1x04-1MP_P1.25mm_Vertical, symbol Connector:Conn_01x04_Socket
- added J11: Extra sensor BOTTOM, Connector_JST:JST_GH_BM04B-GHS-TBT_1x04-1MP_P1.25mm_Vertical, symbol Connector:Conn_01x04_Socket
- added J2: Conn_01x02, 250-202:P-250-202, symbol Connector_Generic:Conn_01x02
- added J7: ToF sensor, Connector_JST:JST_GH_BM04B-GHS-TBT_1x04-1MP_P1.25mm_Vertical, symbol Connector:Conn_01x04_Socket
- added J8: LED, Connector_JST:JST_GH_BM04B-GHS-TBT_1x04-1MP_P1.25mm_Vertical, symbol Connector:Conn_01x04_Socket
- added J9: PWRCONN, Connector_JST:JST_GH_BM03B-GHS-TBT_1x03-1MP_P1.25mm_Vertical, symbol Connector:Conn_01x04_Socket
- added JBUTT1: Conn_01x02, Connector_PinHeader_2.54mm:PinHeader_1x02_P2.54mm_Vertical, symbol Connector_Generic:Conn_01x02
- added L2: 2.2uH, Inductor_SMD:L_0805_2012Metric, symbol Device:L_Small
- added R4, R7: 4.7k, Resistor_SMD:R_0805_2012Metric, symbol Device:R
- added U1: XIAO-ESP32-S3-Plus-SMD, New_XIAO_Series_Footprints:XIAO-ESP32-S3-Plus-SMD, symbol Seeed_Studio_XIAO_Series:XIAO-ESP32-S3 Plus-SMD
- added U5: TPS62163DSG, Package_SON:WSON-8-1EP_2x2mm_P0.5mm_EP0.9x1.6mm_ThermalVias, symbol Regulator_Switching:TPS62162DSG
- added U6: SN74LVC1T45DBV, Package_TO_SOT_SMD:SOT-23-6, symbol Logic_LevelTranslator:SN74LVC1T45DBV
- added U7: BMP388, BMP388:XDCR_BMP388, symbol BMP388:BMP388
Connections:
- net +3V3 is gone; now on net +3.3V: J5.4 (Pin_4)
- net MAIN is gone; now on net +12V: J5.1 (Pin_1)
- net +12V: now also J4.5, C10.1, C11.1, C9.1, D2.C, J2.L1 (Pin_1), J9.2 (Pin_2), JBUTT1.1 (Pin_1), JBUTT1.2 (Pin_2), U5.2 (VIN), U5.3 (EN); no longer J4.1
- net +3.3V: now also C13.1, J10.4 (Pin_4), J11.4 (Pin_4), J7.4 (Pin_4), R4.1, R7.2, U1.12 (3V3), U6.1 (VCCA), U6.5 (DIR), U7.1 (VDDIO), U7.5 (SDO), U7.6 (CSB)
- net ANT: now also J1.1 (In)
- net DIR: now also J4.3, U1.2 (GPIO2_A1_D1); no longer J4.4
- net FEEDBACK: now also J4.4, U1.3 (GPIO3_A2_D2); no longer J4.5
- net GND: now also C10.2, C11.2, C12.1, C13.2, C14.1, C9.2, D2.A, J1.2 (Ext), J1.3 (GND), J1.4 (GND), J1.5 (GND), J10.1 (Pin_1), J11.1 (Pin_1), J2.L2 (Pin_2), J7.1 (Pin_1), J8.2 (Pin_2), J9.1 (Pin_1), J9.3 (Pin_3), U1.13 (GND), U1.34 (PAD), U5.1 (PGND), U5.4 (AGND), U5.5 (FB), U5.9 (PAD), U6.2 (GND), U7.3 (VSS), U7.8 (VSS), U7.9 (VSS)
- net INT: now also U1.8 (GPIO44_D7_RX)
- net MISO: now also U1.10 (GPIO8_A9_D9_MISO)
- net MOSI: now also U1.11 (GPIO9_A10_D10_MOSI)
- net NSS: now also U1.7 (GPIO43_D6_TX)
- net PWM: now also J4.1, U1.1 (GPIO1_A0_D0); no longer J4.3
- net SCK: now also U1.9 (GPIO7_A8_D8_SCK)
- net SCL renamed BMPSCL
- net BMPSCL: now also J10.3 (Pin_3), J11.3 (Pin_3), J7.3 (Pin_3), R4.2, U1.6 (GPIO6_A5_D5_SCL), U7.2 (SCK)
- net SDA renamed BMPSDA
- net BMPSDA: now also J10.2 (Pin_2), J11.2 (Pin_2), J7.2 (Pin_2), R7.1, U1.5 (GPIO5_A4_D4_SDA), U7.4 (SDI)
- new net: C14.2, U7.10 (VDD)
- new net: L2.1, U5.7 (SW)
- new net +5V: C12.2, J8.1 (Pin_1), L2.2, U5.6 (VOS), U6.6 (VCCB)
- new net DIN: J8.3 (Pin_3), U6.4 (B)
- new net LEDSERIAL: U1.21 (GPIO11_DVP_Y8_SPI_MOSI1), U6.3 (A)
- new net STAT: U1.4 (GPIO4_A3_D3)
- no-connect marks 8 -> 29
Other:
- moved on the sheet: D1, R3
